Commit message: Changes

File: src/neo_simulation/robots/mmo_500/urdf/kinect.urdf.xacro (robot description, xacro)
@@ -31,5 +31,5 @@
         <origin xyz="0 0 0" rpy="0 0 ${M_PI/2}"/>
         <geometry>
-          <mesh filename="package://autlab5/urdf/meshes/kinect.dae"/>
+          <mesh filename="package://neo_simulation/robots/mmo_500/meshes/kinect.dae"/>
         </geometry>
       </visual>
